File: hardware/Argus-RPI-HAT.kicad_pcb (KiCad board)
At the start: 4 copper layers, 65 x 56 mm, 75 parts, among them J1 USB_C_Receptacle_USB2.0_16P, J2 GPIO, J3 J_DEBUG, J4 Conn_Coaxial, Q1 2N7002, Q2 2N7002, SW1 SW_RESET, SW2 SW_BOOT, U1 MAX-M10S, U2 ESP32-C6-MINI-1, U3 CAT24C32, U4 AP63203WU, U5 SN74LVC1G125DBV, U6 SN74LVC1G125DBV

Commit message: Add completed KiCad layout, schematics, and brief README
Parts:
- J1: footprint Connector_USB:USB_C_Receptacle_HRO_TYPE-C-31-M-12 -> Argus_Custom:USB_C_HRO_TYPE-C-31-M-12_EdgeSilk
- U2: footprint RF_Module:ESP32-C6-MINI-1 -> Argus_Custom:ESP32-C6-MINI-1_EdgeSilk
- moved R7 15.3 mm to (140.4, 57.2), turned to 90 degrees
- moved R8 12.2 mm to (142.0, 57.2), turned to 90 degrees
- moved TP8 4.92 mm to (156.0, 72.8)
- moved TP9 4.41 mm to (155.8, 61.9)
- moved L1 2.77 mm to (106.2, 61.8), turned to 90 degrees
- moved C9 0.91 mm to (106.0, 59.5), turned to 0 degrees
Routing:
- net GND: track 0.00 -> 163.1 mm, vias 0 -> 18
- net PI_3V3: track 0.00 -> 92.9 mm, vias 0 -> 6
- net /esp32_supervisor/ESP_EN: track 0.00 -> 75.4 mm, vias 0 -> 4
- net /esp32_supervisor/ESP_BOOT: track 0.00 -> 72.5 mm, vias 0 -> 3
- net /esp32_supervisor/ESP_UART_RX: track 0.00 -> 60.1 mm, vias 0 -> 2
- net /esp32_supervisor/ESP_IO2: track 0.00 -> 52.3 mm, vias 0 -> 2
- net PI_UART_RX: track 0.00 -> 50.6 mm, vias 0 -> 1
- net PI_HEARTBEAT: track 0.00 -> 50.3 mm, vias 0 -> 2
- net ESP_GNSS_TX: track 0.00 -> 47.4 mm, vias 0 -> 3
- net /esp32_supervisor/ESP_U0_RX: track 0.00 -> 43.3 mm, vias 0 -> 1
- net /esp32_supervisor/ESP_U0_TX: track 0.00 -> 41.8 mm, vias 0 -> 1
- net /esp32_supervisor/ESP_IO1: track 0.00 -> 39.6 mm, vias 0 -> 2
- net GNSS_TIMEPULSE: track 0.00 -> 37.7 mm, vias 0 -> 3
- net GNSS_RESET_N: track 0.00 -> 33.7 mm, vias 0 -> 2
- net ESP_GNSS_RX: track 0.00 -> 32.5 mm, vias 0 -> 2
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- added copper zone on In2.Cu, net +3V3_ESP
- added copper zone on B.Cu, net GND
- added copper zone on F.Cu, net GND
- added copper zone on In1.Cu, net GND
