File: hardware/Argus-RPI-HAT.kicad_sch (KiCad schematic)
At the start: 49 parts, among them J1 USB_C_Receptacle_USB2.0_16P, J3 J_DEBUG, Q1 2N7002, Q2 2N7002, SW1 SW_RESET, SW2 SW_BOOT, U2 ESP32-C6-MINI-1, U4 AP63203WU, U5 SN74LVC1G125DBV, U6 SN74LVC1G125DBV

Commit message: Add completed KiCad layout, schematics, and brief README
Parts:
- removed C10, C11: 22uF, Capacitor_SMD:C_1206_3216Metric, symbol Device:C_Small
- removed C13, C14, C3, C4: 100nF, Capacitor_SMD:C_0603_1608Metric, symbol Device:C_Small
- removed C2: 10uF, Capacitor_SMD:C_0603_1608Metric, symbol Device:C_Small
- removed C5: 10uF, Capacitor_SMD:C_0805_2012Metric, symbol Device:C_Small
- removed C6: 1uF, Capacitor_SMD:C_0603_1608Metric, symbol Device:C_Small
- removed D1: USBLC6-2SC6, Package_TO_SOT_SMD:SOT-23-6, symbol Power_Protection:USBLC6-2SC6
- removed J1: USB_C_Receptacle_USB2.0_16P, Connector_USB:USB_C_Receptacle_HRO_TYPE-C-31-M-12, symbol Connector:USB_C_Receptacle_USB2.0_16P
- removed J3: J_DEBUG, Connector_PinHeader_2.54mm:PinHeader_1x06_P2.54mm_Vertical, symbol Connector_Generic:Conn_01x06
- removed L2: 3.9uH, Argus_Custom:L_Wurth_WE-PD2SR-7850, symbol Device:L
- removed Q1, Q2: 2N7002, Package_TO_SOT_SMD:SOT-23, symbol Transistor_FET:2N7002
- removed R1, R13, R23, R3, R4: 10K, Resistor_SMD:R_0603_1608Metric, symbol Device:R_US
- removed R10, R9: 5.1K, Resistor_SMD:R_0603_1608Metric, symbol Device:R_US
- removed R12, R2: 100K, Resistor_SMD:R_0603_1608Metric, symbol Device:R_US
- removed R14: 0, Resistor_SMD:R_0603_1608Metric, symbol Device:R_US
- removed R6: 470, Resistor_SMD:R_0603_1608Metric, symbol Device:R_US
- removed R7, R8: 22, Resistor_SMD:R_0603_1608Metric, symbol Device:R_US
- removed SW1: SW_RESET, Button_Switch_SMD:SW_SPST_TL3305A, symbol Switch:SW_Push
- removed SW2: SW_BOOT, Button_Switch_SMD:SW_SPST_TL3305A, symbol Switch:SW_Push
- removed TP1: 3V3, TestPoint:TestPoint_Pad_D1.5mm, symbol Connector:TestPoint
- removed TP10: HEARTBEAT, TestPoint:TestPoint_Pad_D1.5mm, symbol Connector:TestPoint
- removed TP11: SUPERVISOR, TestPoint:TestPoint_Pad_D1.5mm, symbol Connector:TestPoint
- removed TP12: SHUTDOWN, TestPoint:TestPoint_Pad_D1.5mm, symbol Connector:TestPoint
- removed TP15: GNSS_RX, TestPoint:TestPoint_Pad_D1.5mm, symbol Connector:TestPoint
- removed TP16: GNSS_TX, TestPoint:TestPoint_Pad_D1.5mm, symbol Connector:TestPoint
- removed TP17: GNSS_PPS, TestPoint:TestPoint_Pad_D1.5mm, symbol Connector:TestPoint
- removed TP2: GND, TestPoint:TestPoint_Pad_D1.5mm, symbol Connector:TestPoint
- removed TP3: BOOT, TestPoint:TestPoint_Pad_D1.5mm, symbol Connector:TestPoint
- removed TP4: EN, TestPoint:TestPoint_Pad_D1.5mm, symbol Connector:TestPoint
- removed TP5: ESP_RX, TestPoint:TestPoint_Pad_D1.5mm, symbol Connector:TestPoint
- removed TP6: ESP_TX, TestPoint:TestPoint_Pad_D1.5mm, symbol Connector:TestPoint
- removed TP7: VBUS, TestPoint:TestPoint_Pad_D1.5mm, symbol Connector:TestPoint
- removed TP8: D_N, TestPoint:TestPoint_Pad_D1.5mm, symbol Connector:TestPoint
- removed TP9: D_P, TestPoint:TestPoint_Pad_D1.5mm, symbol Connector:TestPoint
- removed U2: ESP32-C6-MINI-1, RF_Module:ESP32-C6-MINI-1, symbol RF_Module:ESP32-C6-MINI-1
- removed U4: AP63203WU, Package_TO_SOT_SMD:TSOT-23-6, symbol Regulator_Switching:AP63203WU
- removed U5, U6: SN74LVC1G125DBV, Package_TO_SOT_SMD:SOT-23-5, symbol 74xGxx:SN74LVC1G125DBV
Connections:
- no-connect marks 10 -> 0
Other:
- added sheet esp32_supervisor (esp32_supervisor.kicad_sch)
- added sheet gnss (gnss.kicad_sch)
- added sheet hat_id_eeprom (hat_id_eeprom.kicad_sch)
- added sheet pi_interface (pi_interface.kicad_sch)
- note removed: "Additional pin functions: https://pinout.xyz/"
- title: (none) -> Argus Raspberry Pi HAT
